File: kicad/vectrix-vehicleman-0.kicad_pcb (KiCad board)
At the start: 2 copper layers, 105.4 x 196.3 mm, 419 parts, among them CN1 SHOU-HAN-TYPE-C16PIN_C393939, J1 Screw_Terminal_01x02, J10 GPS U.FL, J11 LTE U.FL, J12 18650-holder, J17 SW1, J18 SW2, J19 SW3, J20 SW4, J21 Conn_01x07_Pin, J22 CAN 0, J23 PWR_OUT, J24 PWR, J25 K1, J26 K1, J27 K2, J28 K2, J3 CAN 0, J5 CAN SPI1, J6 CAN SPI2, J8 SIM_Card_Shielded, J9 CP PP, K1 G2RL-24 DC5, K2 G2RL-24 DC5, Q1 BSS138, Q10 BSS138-7-F, Q11 BSS138-7-F, Q12 MMBT3904, Q13 MMBT3904, Q14 MMBT3904, Q15 MMBT3904, Q16 Q_NPN_BEC, Q17 Q_NPN_BEC, Q18 MMBT3904, Q19 PMOS_30V_5.5A, Q2 BSS138, Q20 PMOS_30V_5.5A, Q21 PMOS_30V_5.5A, Q22 PMOS_30V_5.5A, Q3 AO3400A, Q4 Q_PMOS_30V_5.5A_SOT23, Q5 BSS138-7-F, Q6 PMOS_30V_5.5A, Q7 N-Fet_Dual_NM8205_SOT23-6, Q8 PMOS_30V_5.5A, Q9 BSS138-7-F, SW1 SW_Push, SW2 SW_DIP_x04, U1 ESP32-WROOM-32E-R2, U10 CH340C, U11 Battery-protector-DW01, U12 HDC1080, U13 MCP2515-xST, U14 MCP2515-xST, U15 SN65HVD231, U16 TPS3808DBV, U17 SN65HVD231, U18 SIM7070G, U19 BOOSTER_2A_12V_MAX_FP6291LR-G1, U2 TPS61022, U20 LM321, U21 DS1307Z+, U22 MCP23017_SO, U23 ME6217C33M5G, U3 TPS62A02DRL, U38 PC817B, U4 TPS563300, U5 TP4056-42-ESOP8, U6 SN65HVD231, U8 LIS3DH, U9 LSM6DS3, Y2 8M, Y3 8M, Y4 Crystal

Commit message: WIP
Parts:
- removed C85, C86: 100nF 50V, Capacitor_SMD:C_0603_1608Metric
- removed D33, D34, D35, D36: 1N4001, Diode_SMD:D_SMA
- removed F42: 200mA PTC, Fuse:Fuse_0805_2012Metric
- removed the H1 at (46.5, 117.2)
- removed the H1 at (46.5, 51.5)
- removed the H2 at (46.5, 107.4)
- removed the H2 at (46.5, 173.2)
- removed the H3 at (130.3, 117.3)
- removed the H3 at (130.3, 51.5)
- removed the H4 at (140.5, 107.4)
- removed the H4 at (140.5, 173.2)
- removed R165, R166, R168, R169: 470R 0603, Resistor_SMD:R_0603_1608Metric
- added C100: Tant 47u 17V, Capacitor_Tantalum_SMD:CP_EIA-3528-12_Kemet-T, F.Cu at (82.5, 235.9)
- added J29: TX RX G, Connector_PinHeader_1.27mm:PinHeader_1x03_P1.27mm_Vertical, F.Cu at (99.1, 234.4)
- added R125: 0R 0603, Resistor_SMD:R_0603_1608Metric, F.Cu at (113.4, 142.0)
- added R126: 0R 0603, Resistor_SMD:R_0603_1608Metric, F.Cu at (120.0, 139.7)
- added R127: 4k7 0603, Resistor_SMD:R_0603_1608Metric, F.Cu at (110.3, 177.7)
- added R145: 4k7 0603, Resistor_SMD:R_0603_1608Metric, F.Cu at (102.7, 150.7)
- added R50: 4k7 0603, Resistor_SMD:R_0603_1608Metric, F.Cu at (103.4, 159.3)
- added R51: 4k7 0603, Resistor_SMD:R_0603_1608Metric, F.Cu at (119.7, 173.2)
- C70: value 100uF 25V -> Tant 47u 17V; footprint Capacitor_SMD:CP_Elec_6.3x7.7 -> Capacitor_Tantalum_SMD:CP_EIA-3528-12_Kemet-T
- F16: value Polyfuse 250V 3A -> Polyfuse 250V .4A
- J21: footprint Connector_PinHeader_1.27mm:PinHeader_1x07_P1.27mm_Vertical -> Connector_PinHeader_1.27mm:PinHeader_1x03_P1.27mm_Vertical
- moved H11 553.5 mm to (46.5, 51.5)
- moved H12 541.3 mm to (46.5, 107.4)
- moved H10 532.3 mm to (46.5, 117.2)
- moved H5 509.6 mm to (46.5, 173.2)
- moved F9 458.9 mm to (101.4, 90.9)
- moved H6 456.4 mm to (130.3, 51.5)
- moved D8 454.8 mm to (107.3, 95.9)
- moved H8 443.4 mm to (130.3, 117.3)
- moved H9 441.1 mm to (140.5, 107.4)
- moved H7 423.1 mm to (140.5, 173.2)
- moved C78 391.0 mm to (66.9, 191.8), turned to -90 degrees
- moved R40 387.0 mm to (97.5, 198.2), turned to -90 degrees
- moved PF2 384.1 mm to (77.2, 172.8)
- moved R41 383.5 mm to (101.4, 200.5), turned to 180 degrees
- moved J21 381.8 mm to (76.1, 175.6), turned to 90 degrees
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Connections:
- C14 pad 2: +5VD -> +3V3
- C60 pad 1: Net-(C60-Pad1) -> +3V3
- C61 pad 1: Net-(C60-Pad1) -> +3V3
- C66 pad 1: Net-(C66-Pad1) -> +3V3
- C67 pad 1: Net-(C66-Pad1) -> +3V3
- D26 pad 1: /LTE/SIM_RST -> Net-(D26A-K1)
- D26 pad 3: /LTE/SIM_CLK -> Net-(D26B-K2)
- D26 pad 5: /LTE/SIM_VDD -> Net-(D26D-K4)
- J21 pad 3: Net-(J21-Pin_3) -> GND
- J8 pad 1: Net-(J8-VCC) -> Net-(D26D-K4)
- J8 pad 2: Net-(J8-RST) -> Net-(D26A-K1)
- J8 pad 3: Net-(J8-CLK) -> Net-(D26B-K2)
- Q18 pad 2: LTE_GPIO5 -> /LTE/LTE_GPIO5
- Q18 pad 3: LTE_GPIO5 -> LTE_GPIO5_HV
- R133 pad 2: LTE_GPIO5 -> LTE_GPIO5_HV
- R134 pad 2: LTE_GPIO5 -> /LTE/LTE_GPIO5
- R135 pad 1: LTE_GPIO5 -> /LTE/LTE_GPIO5
- R167 pad 1: Net-(J21-Pin_4) -> Net-(J21-Pin_2)
- R8 pad 1: Net-(J8-VCC) -> Net-(D26D-K4)
- R96 pad 1: Net-(J8-RST) -> Net-(D26A-K1)
- R97 pad 1: Net-(J8-CLK) -> Net-(D26B-K2)
- U14 pad 13: SPI_CAN1_INT -> SPI_CAN2_INT
- U14 pad 19: SPI_CAN1_RST -> SPI_CAN2_RST
- U18 pad 48: LTE_GPIO5 -> /LTE/LTE_GPIO5
- U21 pad 8: +5VD -> +3V3
- U22 pad 27: Net-(U22-GPA6) -> SPI_CAN1_RST
- U22 pad 28: Net-(U22-GPA7) -> SPI_CAN2_RST
- U22 pad 5: LTE_GPIO5 -> LTE_GPIO5_HV
- U22 pad 6: Net-(U22-GPB5) -> SPI_CAN2_INT
- U22 pad 7: Net-(U22-GPB6) -> SPI_CAN1_INT
- U6 pad 1: CAN_TWAI_TX -> Net-(U6-D)
- U6 pad 4: CAN_TWAI_RX -> Net-(U6-R)
Other:
- board size 105.4 x 196.3 mm -> 105.4 x 197.9 mm
- board text added: "GPS ANT"
- board text added: "TX|RX|G"
