File: kicad/Alarm.kicad_sch (KiCad schematic)
At the start: 0 parts

Commit message: WIP
Parts:
- added C20, C21: 10u 50V, Capacitor_SMD:C_1206_3216Metric, symbol Device:C
- added C48, C49, C50: 100nF 50V, Capacitor_SMD:C_0603_1608Metric, symbol Device:C
- added R40, R41: 4k7 0603, Resistor_SMD:R_0603_1608Metric, symbol Device:R
- added U12: HDC1080, Package_SON:Texas_PWSON-N6, symbol Sensor_Humidity:HDC1080
- added U8: LIS3DH, Package_LGA:LGA-16_3x3mm_P0.5mm_LayoutBorder3x5y, symbol Sensor_Motion:LIS3DH
- added U9: LSM6DS3, Package_LGA:LGA-14_3x2.5mm_P0.5mm_LayoutBorder3x4y, symbol Sensor_Motion:LSM6DS3
Connections:
- new net +3V3: C20.1, C21.1, C48.1, C49.1, C50.1, R40.1, R41.1, U12.5 (VCC), U8.1 (VDD_IO), U8.14 (VDD), U8.7 (SDO), U8.8 (CS), U9.1 (SDO/SA0), U9.12 (CS), U9.2 (SDX), U9.3 (SCX), U9.5 (VDDIO), U9.8 (VDD)
- new net ACCEL_INT: U8.11 (INT1), U9.4 (INT1)
- new net GND: C20.2, C21.2, C48.2, C49.2, C50.2, U12.2 (GND), U8.10 (GND), U8.12 (GND), U8.13 (ADC3), U8.15 (ADC2), U8.16 (ADC1), U8.5 (GND), U9.6 (GND), U9.7 (GND)
- new net I2C_SDA: R40.2, U12.1 (SDA), U8.6 (SDI), U9.14 (SDA)
- new net I2C_SLC: R41.2, U12.6 (SCL), U8.4 (SPC), U9.13 (SCL)
- no-connect marks 0 -> 2
Other:
- note added: "ACCEL"
- note added: "GYRO"
- note added: "TEMP/HUMIDITY"

Commit message: sch done-ish
Other:
- company: (none) -> ©CC-BY-NC
- title: (none) -> VehicleMan
Changed lines of the file:
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@@
 	(generator_version "9.0")
 	(paper "A4")
+	(title_block
+		(title "VehicleMan")
+		(date "2025-03-04")
+		(rev "0")
+		(company "©CC-BY-NC")
+	)
 	(text "ACCEL"
 		(exclude_from_sim no)

Commit message: R0
Parts:
- added D33, D34: 1N4148W, Diode_SMD:D_SOD-123, symbol Diode:1N4148
Connections:
- net ACCEL_INT: now also D33.1 (K), D34.1 (K); no longer U8.11 (INT1), U9.4 (INT1)
- new net ACCEL_PD_INT: D34.2 (A), U8.11 (INT1)
- new net GYRO_INT: D33.2 (A), U9.4 (INT1)
