File: kicad/CAN.kicad_sch (KiCad schematic)
At the start: 1 part, among them U6 SN65HVD231

Commit message: WIP
Parts:
- added C51, C54, C61, C66, C69: 100nF 50V, Capacitor_SMD:C_0603_1608Metric, symbol Device:C
- added C52, C53, C60, C67, C68: 10u 50V, Capacitor_SMD:C_1206_3216Metric, symbol Device:C
- added C55, C56, C62, C65: 20pF 50V, Capacitor_SMD:C_0603_1608Metric, symbol Device:C
- added R42, R44, R52, R53, R54, R55, R56, R66: 10k 0603, Resistor_SMD:R_0603_1608Metric, symbol Device:R
- added R45, R65: 4k7 0603, Resistor_SMD:R_0603_1608Metric, symbol Device:R
- added R57, R58, R59, R60, R61, R62, R63, R64: 0R 0603, Resistor_SMD:R_0603_1608Metric, symbol Device:R
- added U13, U14: MCP2515-xST, Package_SO:TSSOP-20_4.4x6.5mm_P0.65mm, symbol Interface_CAN_LIN:MCP2515-xST
- added U15, U17: SN65HVD231, Package_SO:SOIC-8_3.9x4.9mm_P1.27mm, symbol Interface_CAN_LIN:SN65HVD231
- added Y2, Y3: 8M, Crystal:Crystal_HC49-U_Horizontal, symbol Device:Crystal
Connections:
- net GND: now also C51.2, C52.2, C53.2, C54.2, C55.1, C56.2, C60.2, C61.2, C62.2, C65.1, C66.2, C67.2, C68.2, C69.2, R42.2, R44.2, R66.2, U13.10 (VSS), U14.10 (VSS), U15.2 (GND), U17.2 (GND)
- net CAN_TWAI_TX: now reaches U6.1 (D)
- net +3V3: now reaches U6.3 (VCC)
- net +3V3: now also C51.1, C52.1, C53.1, C54.1, C68.1, C69.1, R45.1, R52.1, R53.1, R54.1, R55.1, R56.1, R65.1, U13.20 (VDD), U14.20 (VDD), U15.3 (VCC), U17.3 (VCC)
- net CAN_TWAI_RX: now reaches U6.4 (R)
- net CAN_L_TWAI: now reaches U6.6 (CANL)
- net CAN_H_TWAI: now reaches U6.7 (CANH)
- net at U6.8 (Rs): now also R42.1
- new net: R45.2, U13.2 (RXCAN), U15.4 (R)
- new net: C55.2, U13.9 (OSC1), Y2.1
- new net: R61.2, U14.16 (SI)
- new net: R65.2, U14.2 (RXCAN), U17.4 (R)
- new net: C56.1, U13.8 (OSC2), Y2.2
- new net: C66.1, C67.1
- new net: R44.1, U15.8 (Rs)
- new net: U13.1 (TXCAN), U15.1 (D)
- new net: R60.2, U13.14 (SCK)
- new net: R57.2, U13.16 (SI)
- new net: R58.2, U13.17 (SO)
- new net: R59.2, U13.18 (~{CS})
- new net: R66.1, U17.8 (Rs)
- new net: U14.1 (TXCAN), U17.1 (D)
- new net: R64.2, U14.14 (SCK)
- new net: R62.2, U14.17 (SO)
- new net: R63.2, U14.18 (~{CS})
- new net: C62.1, U14.8 (OSC2), Y3.2
- new net: C65.2, U14.9 (OSC1), Y3.1
- new net: C60.1, C61.1
- new net CAN_H_SPI_1: U15.7 (CANH)
- new net CAN_H_SPI_2: U17.7 (CANH)
- new net CAN_L_SPI_1: U15.6 (CANL)
- new net CAN_L_SPI_2: U17.6 (CANL)
- new net SPI_CAN1_INT: U13.13 (~{INT}), U14.13 (~{INT})
- new net SPI_CAN1_RST: U13.19 (~{RESET}), U14.19 (~{RESET})
- new net VSPI_CAN1_CS: R55.2, R59.1
- new net VSPI_CAN2_CS: R56.2, R63.1
- new net VSPI_MISO: R53.2, R58.1, R62.1
- new net VSPI_MOSI: R54.2, R57.1, R61.1
- new net VSPI_SCK: R52.2, R60.1, R64.1
- no-connect marks 0 -> 15
Other:
- note added: "CAN SPI1 TRANSCV"
- note added: "CAN TWAI TRANSCV"
- moved on the sheet: U6

Commit message: sch done-ish
Parts:
- added R94, R95: 4k7 0603, Resistor_SMD:R_0603_1608Metric, symbol Device:R
Connections:
- net VSPI_CAN1_CS: now also R94.2
- net VSPI_CAN2_CS: now also R95.2
- net at C66.1, C67.1: now also R95.1
- net at C60.1, C61.1: now also R94.1
Other:
- note added: "CAN SPI2 TRANSCV"
- company: (none) -> ©CC-BY-NC
- title: (none) -> VehicleMan
- moved on the sheet: C51, C52, C53, C54, C55, C56, C60, C61, C62, C65, C66, C67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

Commit message: WIP
Parts:
- removed R94, R95: 4k7 0603, Resistor_SMD:R_0603_1608Metric, symbol Device:R
- Y2, Y3: footprint Crystal:Crystal_HC49-U_Horizontal -> Crystal:Crystal_SMD_HC49-SD
Changed lines of the file:
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@@
 	)
 	(junction
-		(at 74.93 132.08)
-		(diameter 0)
-		(color 0 0 0 0)
-	)
-	(junction
 		(at 44.45 179.07)
 		(diameter 0)
@@
 	)
 	(junction
-		(at 30.48 156.21)
-		(diameter 0)
-		(color 0 0 0 0)
-	)
-	(junction
 		(at 100.33 80.01)
 		(diameter 0)
@@
 	)
 	(junction
-		(at 30.48 85.09)
-		(diameter 0)
-		(color 0 0 0 0)
-	)
-	(junction
 		(at 87.63 45.72)
 		(diameter 0)
@@
 	)
 	(junction
-		(at 74.93 60.96)
-		(diameter 0)
-		(color 0 0 0 0)
-	)
-	(junction
 		(at 59.69 22.86)
 		(diameter 0)
@@
 	(wire
 		(pts
-			(xy 30.48 156.21) (xy 53.34 156.21)
-		)
-		(stroke
-			(width 0)
-			(type default)
-		)
-	)
-	(wire
-		(pts
 			(xy 60.96 153.67) (xy 63.5 153.67)
 		)
@@
 	(wire
 		(pts
-			(xy 29.21 85.09) (xy 30.48 85.09)
-		)
-		(stroke
-			(width 0)
-			(type default)
-		)
-	)
-	(wire
-		(pts
 			(xy 119.38 158.75) (xy 121.92 158.75)
 		)
@@
 	(wire
 		(pts
-			(xy 30.48 148.59) (xy 30.48 132.08)
-		)
-		(stroke
-			(width 0)
-			(type default)
-		)
-	)
-	(wire
-		(pts
 			(xy 132.08 92.71) (xy 132.08 95.25)
 		)
@@
 	(wire
 		(pts
-			(xy 30.48 85.09) (xy 53.34 85.09)
+			(xy 29.21 85.09) (xy 53.34 85.09)
 		)
 		(stroke
@@
 	(wire
 		(pts
-			(xy 29.21 156.21) (xy 30.48 156.21)
+			(xy 29.21 156.21) (xy 53.34 156.21)
 		)
 		(stroke
@@
 	(wire
 		(pts
-			(xy 30.48 132.08) (xy 74.93 132.08)
-		)
-		(stroke
-			(width 0)
-			(type default)
-		)
-	)
-	(wire
-		(pts
 			(xy 60.96 82.55) (xy 63.5 82.55)
 		)
@@
 	(wire
 		(pts
-			(xy 30.48 60.96) (xy 74.93 60.96)
-		)
-		(stroke
-			(width 0)
-			(type default)
-		)
-	)
-	(wire
-		(pts
 			(xy 132.08 95.25) (xy 160.02 95.25)
 		)
@@
 	(wire
 		(pts
-			(xy 30.48 77.47) (xy 30.48 60.96)
-		)
-		(stroke
-			(width 0)
-			(type default)
-		)
-	)
-	(wire
-		(pts
 			(xy 114.3 77.47) (xy 114.3 80.01)
 		)
@@
 	)
 	(symbol
-		(lib_id "Device:R")
-		(at 30.48 81.28 0)
-		(mirror y)
-		(unit 1)
-		(exclude_from_sim no)
-		(in_bom yes)
-		(on_board yes)
-		(dnp no)
-		(property "Reference" "R94"
-			(at 27.94 80.0099 0)
-			(effects
-				(font
-					(size 1.27 1.27)
-				)
-				(justify left)
-			)
-		)
-		(property "Value" "4k7 0603"
-			(at 27.94 82.5499 0)
-			(effects
-				(font
-					(size 1.27 1.27)
-				)
-				(justify left)
-			)
-		)
-		(property "Footprint" "Resistor_SMD:R_0603_1608Metric"
-			(at 32.258 81.28 90)
-			(effects
-				(font
-					(size 1.27 1.27)
-				)
-				(hide yes)
-			)
-		)
-		(property "Datasheet" "~"
-			(at 30.48 81.28 0)
-			(effects
-				(font
-					(size 1.27 1.27)
-				)
-				(hide yes)
-			)
-		)
-		(property "Description" "Resistor"
-			(at 30.48 81.28 0)
-			(effects
-				(font
-					(size 1.27 1.27)
-				)
-				(hide yes)
-			)
-		)
-		(property "LCSC" "C99782"
-			(at 30.48 81.28 0)
-			(effects
-				(font
-					(size 1.27 1.27)
-				)
-				(hide yes)
-			)
-		)
-		(pin "1"
-		)
-		(pin "2"
-		)
-		(instances
-			(project "vectrix-vehicleman-0"
-				(path "/05d12b30-c3b1-455d-b907-9e9d56cc8f30/7d8f0b1a-bbaa-47a2-a4c5-01df157da82c"
-					(reference "R94")
-					(unit 1)
-				)
-			)
-		)
-	)
-	(symbol
 		(lib_id "power:GND")
 		(at 49.53 163.83 0)
@@
 	)
 	(symbol
-		(lib_id "Device:R")
-		(at 30.48 152.4 0)
-		(mirror y)
-		(unit 1)
-		(exclude_from_sim no)
-		(in_bom yes)
-		(on_board yes)
-		(dnp no)
-		(property "Reference" "R95"
-			(at 27.94 151.1299 0)
-			(effects
-				(font
-					(size 1.27 1.27)
-				)
-				(justify left)
-			)
-		)
-		(property "Value" "4k7 0603"
-			(at 27.94 153.6699 0)
-			(effects
-				(font
-					(size 1.27 1.27)
-				)
-				(justify left)
-			)
-		)
-		(property "Footprint" "Resistor_SMD:R_0603_1608Metric"
-			(at 32.258 152.4 90)
-			(effects
-				(font
-					(size 1.27 1.27)
-				)
-				(hide yes)
-			)
-		)
-		(property "Datasheet" "~"
-			(at 30.48 152.4 0)
-			(effects
-				(font
-					(size 1.27 1.27)
-				)
-				(hide yes)
-			)
-		)
-		(property "Description" "Resistor"
-			(at 30.48 152.4 0)
-			(effects
-				(font
-					(size 1.27 1.27)
-				)
-				(hide yes)
-			)
-		)
-		(property "LCSC" "C99782"
-			(at 30.48 152.4 0)
-			(effects
-				(font
-					(size 1.27 1.27)
-				)
-				(hide yes)
-			)
-		)
-		(pin "1"
-		)
-		(pin "2"
-		)
-		(instances
-			(project "vectrix-vehicleman-0"
-				(path "/05d12b30-c3b1-455d-b907-9e9d56cc8f30/7d8f0b1a-bbaa-47a2-a4c5-01df157da82c"
-					(reference "R95")
-					(unit 1)
-				)
-			)
-		)
-	)
-	(symbol
 		(lib_id "Interface_CAN_LIN:SN65HVD231")
 		(at 59.69 33.02 0)
@@
 			)
 		)
-		(property "Footprint" "Crystal:Crystal_HC49-U_Horizontal"
+		(property "Footprint" "Crystal:Crystal_SMD_HC49-SD"
 			(at 44.45 104.14 0)
 			(effects
@@
 			)
 		)
-		(property "Footprint" "Crystal:Crystal_HC49-U_Horizontal"
+		(property "Footprint" "Crystal:Crystal_SMD_HC49-SD"
 			(at 44.45 175.26 0)
 			(effects

Commit message: WIP
Parts:
- added R125, R126: 0R 0603, Resistor_SMD:R_0603_1608Metric, symbol Device:R
- added R127, R145, R50, R51: 4k7 0603, Resistor_SMD:R_0603_1608Metric, symbol Device:R
Connections:
- net +3V3: now also C60.1, C61.1, C66.1, C67.1, R127.1, R145.1, R50.1, R51.1
- net CAN_TWAI_RX: now also R126.2; no longer U6.4 (R)
- net CAN_TWAI_TX: now also R125.2; no longer U6.1 (D)
- net SPI_CAN1_INT: now also R145.2; no longer U14.13 (~{INT})
- net SPI_CAN1_RST: now also R50.2; no longer U14.19 (~{RESET})
- new net: R125.1, U6.1 (D)
- new net: R126.1, U6.4 (R)
- new net SPI_CAN2_INT: R127.2, U14.13 (~{INT})
- new net SPI_CAN2_RST: R51.2, U14.19 (~{RESET})

Commit message: bom cleanup
Parts:
- Y2, Y3: Field5 C12674 -> (none); LCSC (none) -> C12674
Changed lines of the file:
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@@
 			)
 		)
-		(property "Field5" "C12674"
+		(property "LCSC" "C12674"
 			(at 44.45 104.14 90)
 			(effects
@@
 			)
 		)
-		(property "Field5" "C12674"
+		(property "LCSC" "C12674"
 			(at 44.45 175.26 90)
 			(effects
