File: kicad/DCDC.kicad_sch (KiCad schematic)
At the start: 30 parts, among them Q3 Q_PMOS_30V_5.5A_SOT23, U2 TPS61022, U3 TPS62A02DRL, U4 TPS563300

Commit message: WIP
Connections:
- net +12V: now also U7.1 (+12V)
- net GND: now also U7.3 (GND)
- no-connect marks 0 -> 1
Other:
- note added: "150-180Vin MAX to 12V DCDC"
- note added: "BATT BOOST TO 4V2"
- note added: "EXT12V TO 4V2"
- note added: "MAIN TO 3V3"
- note added: "SOMETHING OR-ING"
Changed lines of the file:
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@@
 	(generator_version "9.0")
 	(paper "A4")
+	(text "BATT BOOST TO 4V2\n"
+		(exclude_from_sim no)
+		(at 38.354 177.8 0)
+		(effects
+			(font
+				(size 3 3)
+				(thickness 0.6)
+				(bold yes)
+			)
+		)
+	)
+	(text "SOMETHING\nOR-ING\n"
+		(exclude_from_sim no)
+		(at 185.166 149.606 0)
+		(effects
+			(font
+				(size 3 3)
+				(thickness 0.6)
+				(bold yes)
+			)
+		)
+	)
 	(text "https://webench.ti.com/appinfo/webench/scripts/SDP.cgi?ID=62C56A5871A9F317"
 		(exclude_from_sim no)
@@
 		)
 	)
+	(text "MAIN TO 3V3\n"
+		(exclude_from_sim no)
+		(at 39.624 53.34 0)
+		(effects
+			(font
+				(size 3 3)
+				(thickness 0.6)
+				(bold yes)
+			)
+		)
+	)
+	(text "EXT12V TO 4V2\n"
+		(exclude_from_sim no)
+		(at 48.26 130.81 0)
+		(effects
+			(font
+				(size 3 3)
+				(thickness 0.6)
+				(bold yes)
+			)
+		)
+	)
 	(text "https://webench.ti.com/appinfo/webench/scripts/SDP.cgi?ID=FB38C6AE199D341B"
 		(exclude_from_sim no)
@@
 		)
 	)
+	(text "150-180Vin MAX to 12V DCDC"
+		(exclude_from_sim no)
+		(at 177.546 32.258 0)
+		(effects
+			(font
+				(size 3 3)
+				(thickness 0.6)
+				(bold yes)
+			)
+		)
+	)
 	(junction
 		(at 78.74 172.72)
@@
 		(diameter 0)
 		(color 0 0 0 0)
+	)
+	(no_connect
+		(at 173.99 43.18)
 	)
 	(wire
@@
 	)
 	(symbol
+		(lib_id "power:GND")
+		(at 184.15 59.69 0)
+		(unit 1)
+		(exclude_from_sim no)
+		(in_bom yes)
+		(on_board yes)
+		(dnp no)
+		(fields_autoplaced yes)
+		(property "Reference" "#PWR057"
+			(at 184.15 66.04 0)
+			(effects
+				(font
+					(size 1.27 1.27)
+				)
+				(hide yes)
+			)
+		)
+		(property "Value" "GND"
+			(at 184.15 64.77 0)
+			(effects
+				(font
+					(size 1.27 1.27)
+				)
+			)
+		)
+		(property "Footprint" ""
+			(at 184.15 59.69 0)
+			(effects
+				(font
+					(size 1.27 1.27)
+				)
+				(hide yes)
+			)
+		)
+		(property "Datasheet" ""
+			(at 184.15 59.69 0)
+			(effects
+				(font
+					(size 1.27 1.27)
+				)
+				(hide yes)
+			)
+		)
+		(property "Description" "Power symbol creates a global label with name \"GND\" , ground"
+			(at 184.15 59.69 0)
+			(effects
+				(font
+					(size 1.27 1.27)
+				)
+				(hide yes)
+			)
+		)
+		(pin "1"
+		)
+		(instances
+			(project "vectrix-vehicleman-0"
+				(path "/05d12b30-c3b1-455d-b907-9e9d56cc8f30/9caf0d13-589a-469d-9b5c-d69632aa737b"
+					(reference "#PWR057")
+					(unit 1)
+				)
+			)
+		)
+	)
+	(symbol
 		(lib_id "Converter_DCDC:TPS61022")
 		(at 78.74 165.1 0)
@@
 					(unit 1)
 				)
+			)
+		)
+	)
+	(symbol
+		(lib_id "power:+12V")
+		(at 173.99 54.61 90)
+		(unit 1)
+		(exclude_from_sim no)
+		(in_bom yes)
+		(on_board yes)
+		(dnp no)
+		(fields_autoplaced yes)
+		(property "Reference" "#PWR056"
+			(at 177.8 54.61 0)
+			(effects
+				(font
+					(size 1.27 1.27)
+				)
+				(hide yes)
+			)
+		)
+		(property "Value" "+12V"
+			(at 170.18 54.6099 90)
+			(effects
+				(font
+					(size 1.27 1.27)
+				)
+				(justify left)
+			)
+		)
+		(property "Footprint" ""
+			(at 173.99 54.61 0)
+			(effects
+				(font
+					(size 1.27 1.27)
+				)
+				(hide yes)
+			)
+		)
+		(property "Datasheet" ""
+			(at 173.99 54.61 0)
+			(effects
+				(font
+					(size 1.27 1.27)
+				)
+				(hide yes)
+			)
+		)
+		(property "Description" "Power symbol creates a global label with name \"+12V\""
+			(at 173.99 54.61 0)
+			(effects
+				(font
+					(size 1.27 1.27)
+				)
+				(hide yes)
+			)
+		)
+		(pin "1"
+		)
+		(instances
+			(project "vectrix-vehicleman-0"
+				(path "/05d12b30-c3b1-455d-b907-9e9d56cc8f30/9caf0d13-589a-469d-9b5c-d69632aa737b"
+					(reference "#PWR056")
+					(unit 1)
+				)

Commit message: sch done-ish
Parts:
- removed C30: 100nF 50V, Capacitor_SMD:C_0603_1608Metric, symbol Device:C
- removed D8, D9: D_Schottky_5A_360mV@5A, Diode_SMD:D_SOD-128, symbol Skrubis:D_Schottky_3A_40V
- removed Q3: Q_PMOS_30V_5.5A_SOT23, Package_TO_SOT_SMD:SOT-23, symbol Skrubis:Q_PMOS_30V_5.5A_SOT23
- added C72, C73, C83, C84: 100nF 50V, Capacitor_SMD:C_0603_1608Metric, symbol Device:C
- added C74, C82: 10u 50V, Capacitor_SMD:C_1206_3216Metric, symbol Device:C
- added C75: 100uF 25V, Capacitor_SMD:CP_Elec_6.3x7.7, symbol Device:C_Polarized
- added D20, D8, D9: Schottky 40V 10A, Package_TO_SOT_SMD:TO-277B, symbol Device:D_Schottky_AAK
- added D21: D_Schottky_3A_40V, Diode_SMD:D_SMA, symbol Skrubis:D_Schottky_3A_40V
- added FB3: FB_100R_2.5A, Inductor_SMD:L_0603_1608Metric, symbol Skrubis:FB_100R_2.5A
- added L2: Inductor_3.3uH_4.7A_shielded, Inductor_SMD:L_7.3x7.3_H4.5, symbol Skrubis:Inductor_3.3uH_4.7A_shielded
- added Q3: AO3400A, Package_TO_SOT_SMD:SOT-23, symbol Transistor_FET:AO3400A
- added Q6, Q8: PMOS_30V_5.5A, Package_TO_SOT_SMD:SOT-23, symbol Skrubis:Q_PMOS_30V_5.5A_SOT23
- added R108, R109, R110, R111: 0R 0603, Resistor_SMD:R_0603_1608Metric, symbol Device:R
- added R113, R114: 100k 0603, Resistor_SMD:R_0603_1608Metric, symbol Device:R
- added R68: R_47K_0603, Resistor_SMD:R_0603_1608Metric, symbol Skrubis:R_100K_0603
- added R69: 10k 0603, Resistor_SMD:R_0603_1608Metric, symbol Device:R
- added TP20: TP_2mm, TestPoint:TestPoint_Pad_D2.0mm, symbol Connector:TestPoint
- added U19: BOOSTER_2A_12V_MAX_FP6291LR-G1, Package_TO_SOT_SMD:SOT-23-6, symbol Skrubis:BOOSTER_2A_12V_MAX_FP6291LR-G1
- C24: value 22uF 63V -> 100uF 25V; LCSC C267472 -> C2918360
- C26, C28, C29, L4, R10, R11, U2, U7: now not fitted
- C27: value 22uF 63V -> 100uF 25V; LCSC C267472 -> C2918360; now not fitted
- R12: value 10k 0603 -> 100k 0603; LCSC C2930027 -> C14675; now not fitted
- R13: value 0R -> 100k 0603; footprint Resistor_SMD:R_0805_2012Metric -> Resistor_SMD:R_0603_1608Metric; LCSC (none) -> C14675
Connections:
- net +12V: now also D20.3 (K), D8.3 (K), D9.3 (K), R110.2, R111.2; no longer U7.1 (+12V)
- net 4V2-FROM-12V: now also Q6.3 (D), R108.2, R109.2; no longer R12.1, R13.1
- net 4V2-FROM-BAT: now also R12.2, C72.1, Q3.1 (G), Q6.1 (G), Q8.3 (D)
- net GND: now also R12.1, C72.2, C73.2, C74.2, C75.2, C82.2, C83.2, C84.2, Q3.2 (S), R68.2, R69.2, U19.2 (GND); no longer R12.2
- net VBUS: now also R13.2, C82.1, C83.1, C84.1, L2.1, Q6.2 (S), Q8.2 (S), R108.1, R109.1, U19.4 (EN), U19.5 (Vcc)
- new net: R113.2, R114.1
- new net: R114.2, R69.1, U19.3 (FB)
- new net: C73.1, C74.1, C75.1, D21.1 (K), FB3.1, R113.1
- new net: R68.1, U19.6 (OC)
- new net: D21.2 (A), L2.2, U19.1 (LX)
- new net: Q3.3 (D), Q8.1 (G), R13.1
- new net +12P: D9.1 (A), D9.2 (A), R110.1, R111.1
- new net 12V_BATT: D20.1 (A), D20.2 (A), FB3.2, TP20.1
- new net 12V_HV: D8.1 (A), D8.2 (A), U7.1 (+12V)
Other:
- note added: "1A trip"
- note added: "4V2 ORING"
- note added: "BATT BOOST TO 12V"
- note added: "IF EXT PWR EXISTS - USE THAT IF NO EXT PWR EXISTS - USE BATT"
- note added: "ext 12V"
- note added: "https://github.com/kaminaris/GigaESC/tree/master/PowerBoard/TL494V2OC"
- note added: "hv 12v"
- note removed: "SOMETHING OR-ING"
- company: (none) -> ©CC-BY-NC
- title: (none) -> VehicleMan

Commit message: WIP
Parts:
- removed C24, C27: 100uF 25V, Capacitor_SMD:CP_Elec_6.3x7.7, symbol Device:C_Polarized
- removed D8: Schottky 40V 10A, Package_TO_SOT_SMD:TO-277B, symbol Device:D_Schottky_AAK
- removed TP20: TP_2mm, TestPoint:TestPoint_Pad_D2.0mm, symbol Connector:TestPoint
- added C27, C38: 100nF 50V, Capacitor_SMD:C_0603_1608Metric, symbol Device:C
- added C37: 100uF 25V, Capacitor_SMD:CP_Elec_6.3x7.7, symbol Device:C_Polarized
- added C91, C92, C97, C99: 10u 50V, Capacitor_SMD:C_1206_3216Metric, symbol Device:C
- added D41: Schottky 40V 10A, Package_TO_SOT_SMD:TO-277B, symbol Device:D_Schottky_AAK
- added D8: SMAJ18A, Diode_SMD:D_SMA, symbol Diode:SMAJ18A
- added F16: Polyfuse 250V 3A, Fuse:Fuse_Bourns_MF-RHT200, symbol Device:Polyfuse
- added F9: Polyfuse 2A, Fuse:Fuse_2920_7451Metric, symbol Device:Polyfuse
- C83: value 100nF 50V -> 10u 50V; footprint Capacitor_SMD:C_0603_1608Metric -> Capacitor_SMD:C_1206_3216Metric; LCSC C14663 -> C13585
- U7: now fitted
Connections:
- net +12V: now also D41.3 (K)
- net +3V3: now also C37.1, C38.1
- net +BATT: now also C27.1
- net 12V_HV: now also D41.1 (A), D41.2 (A), F9.1; no longer U7.1 (+12V)
- net 4V2-FROM-12V: now also C97.1, C99.1
- net 4V2-FROM-BAT: now also C91.1, C92.1
- net GND: now also C27.2, C37.2, C38.2, C91.2, C92.2, C97.2, C99.2, D8.2 (A2)
- net +VDC: no longer names the net of U7.2 (HV)
- net +VDC: now also F16.2
- new net: D8.1 (A1), F9.2, U7.1 (+12V)
- new net HV+: F16.1
Other:
- note removed: "150-180Vin MAX to 12V DCDC"
- note removed: "hv 12v"
- moved on the sheet: C25

Commit message: WIP
Parts:
- F16: value Polyfuse 250V 3A -> Polyfuse 250V .4A; LCSC C369126 -> C693579
Changed lines of the file:
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@@
 			)
 		)
-		(property "Value" "Polyfuse 250V 3A"
+		(property "Value" "Polyfuse 250V .4A"
 			(at 177.8 52.07 90)
 			(effects
@@
 			)
 		)
-		(property "LCSC" "C369126"
+		(property "LCSC" "C693579"
 			(at 177.8 55.88 90)
 			(effects

Commit message: R0
Parts:
- removed R110, R111: 0R 0603, Resistor_SMD:R_0603_1608Metric, symbol Device:R
- added JP1, JP7: SolderJumper_2_Open, Jumper:SolderJumper-2_P1.3mm_Open_Pad1.0x1.5mm, symbol Jumper:SolderJumper_2_Open
- D8, F16, F9, U7: now not fitted
Connections:
- net +12P: now also JP1.2 (B), JP7.2 (B)
- net +12V: now also JP1.1 (A), JP7.1 (A)
Changed lines of the file:
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@@
 	)
 	(junction
-		(at 53.34 125.73)
+		(at 271.78 222.25)
 		(diameter 0)
 		(color 0 0 0 0)
 	)
 	(junction
-		(at 271.78 222.25)
+		(at 53.34 125.73)
 		(diameter 0)
 		(color 0 0 0 0)
@@
 	)
 	(junction
+		(at 276.86 222.25)
+		(diameter 0)
+		(color 0 0 0 0)
+	)
+	(junction
 		(at 114.3 214.63)
 		(diameter 0)
@@
 	)
 	(junction
-		(at 276.86 222.25)
-		(diameter 0)
-		(color 0 0 0 0)
-	)
-	(junction
 		(at 217.17 138.43)
 		(diameter 0)
@@
 	(wire
 		(pts
+			(xy 276.86 222.25) (xy 290.83 222.25)
+		)
+		(stroke
+			(width 0)
+			(type default)
+		)
+	)
+	(wire
+		(pts
 			(xy 38.1 214.63) (xy 40.64 214.63)
 		)
@@
 	(wire
 		(pts
-			(xy 276.86 222.25) (xy 290.83 222.25)
-		)
-		(stroke
-			(width 0)
-			(type default)
-		)
-	)
-	(wire
-		(pts
 			(xy 101.6 167.64) (xy 101.6 165.1)
 		)
@@
 	(wire
 		(pts
+			(xy 271.78 222.25) (xy 276.86 222.25)
+		)
+		(stroke
+			(width 0)
+			(type default)
+		)
+	)
+	(wire
+		(pts
 			(xy 74.93 55.88) (xy 77.47 55.88)
 		)
@@
 	(wire
 		(pts
-			(xy 271.78 222.25) (xy 276.86 222.25)
-		)
-		(stroke
-			(width 0)
-			(type default)
-		)
-	)
-	(wire
-		(pts
 			(xy 92.71 55.88) (xy 95.25 55.88)
 		)
@@
 	)
 	(symbol
-		(lib_id "Device:R")
-		(at 276.86 218.44 0)
-		(mirror y)
-		(unit 1)
-		(exclude_from_sim no)
-		(in_bom yes)
-		(on_board yes)
-		(dnp no)
-		(property "Reference" "R111"
-			(at 276.86 220.218 90)
-			(effects
-				(font
-					(size 1.27 1.27)
-				)
-				(justify left)
-			)
-		)
-		(property "Value" "0R 0603"
-			(at 279.654 220.472 90)
-			(effects
-				(font
-					(size 1.27 1.27)
-				)
-				(justify left)
-			)
-		)
-		(property "Footprint" "Resistor_SMD:R_0603_1608Metric"
-			(at 278.638 218.44 90)
-			(effects
-				(font
-					(size 1.27 1.27)
-				)
-				(hide yes)
-			)
-		)
-		(property "Datasheet" "~"
-			(at 276.86 218.44 0)
-			(effects
-				(font
-					(size 1.27 1.27)
-				)
-				(hide yes)
-			)
-		)
-		(property "Description" "Resistor"
-			(at 276.86 218.44 0)
-			(effects
-				(font
-					(size 1.27 1.27)
-				)
-				(hide yes)
-			)
-		)
-		(property "LCSC" "C21189"
-			(at 276.86 218.44 0)
-			(effects
-				(font
-					(size 1.27 1.27)
-				)
-				(hide yes)
-			)
-		)
-		(pin "2"
-		)
-		(pin "1"
-		)
-		(instances
-			(project "vectrix-vehicleman-0"
-				(path "/05d12b30-c3b1-455d-b907-9e9d56cc8f30/9caf0d13-589a-469d-9b5c-d69632aa737b"
-					(reference "R111")
-					(unit 1)
-				)
-			)
-		)
-	)
-	(symbol
 		(lib_id "Device:L")
 		(at 99.06 55.88 90)
@@
 		(in_bom yes)
 		(on_board yes)
-		(dnp no)
+		(dnp yes)
 		(fields_autoplaced yes)
 		(property "Reference" "F9"
@@
 	)
 	(symbol
-		(lib_id "Device:R")
-		(at 271.78 218.44 0)
-		(mirror y)
-		(unit 1)
-		(exclude_from_sim no)
-		(in_bom yes)
-		(on_board yes)
-		(dnp no)
-		(property "Reference" "R110"
-			(at 271.78 220.218 90)
-			(effects
-				(font
-					(size 1.27 1.27)
-				)
-				(justify left)
-			)
-		)
-		(property "Value" "0R 0603"
-			(at 274.574 220.472 90)
-			(effects
-				(font
-					(size 1.27 1.27)
-				)
-				(justify left)
-			)
-		)
-		(property "Footprint" "Resistor_SMD:R_0603_1608Metric"
-			(at 273.558 218.44 90)
-			(effects
-				(font
-					(size 1.27 1.27)
-				)
-				(hide yes)
-			)
-		)
-		(property "Datasheet" "~"
-			(at 271.78 218.44 0)
-			(effects
-				(font
-					(size 1.27 1.27)
-				)
-				(hide yes)
-			)
-		)
-		(property "Description" "Resistor"
-			(at 271.78 218.44 0)
-			(effects
-				(font
-					(size 1.27 1.27)
-				)
-				(hide yes)
-			)
-		)
-		(property "LCSC" "C21189"
-			(at 271.78 218.44 0)
-			(effects
-				(font
-					(size 1.27 1.27)
-				)
-				(hide yes)
-			)
-		)
-		(pin "2"
-		)
-		(pin "1"
-		)
-		(instances
-			(project "vectrix-vehicleman-0"
-				(path "/05d12b30-c3b1-455d-b907-9e9d56cc8f30/9caf0d13-589a-469d-9b5c-d69632aa737b"
-					(reference "R110")
-					(unit 1)
-				)
-			)
-		)
-	)
-	(symbol
 		(lib_id "power:VBUS")
 		(at 38.1 214.63 0)
@@
 		(in_bom yes)
 		(on_board yes)
-		(dnp no)
+		(dnp yes)
 		(fields_autoplaced yes)
 		(property "Reference" "F16"
@@
 	)
 	(symbol
+		(lib_id "Jumper:SolderJumper_2_Open")
+		(at 271.78 218.44 90)
+		(unit 1)
+		(exclude_from_sim no)
+		(in_bom no)
+		(on_board yes)
+		(dnp no)
+		(property "Reference" "JP1"
+			(at 262.89 230.632 90)
+			(effects
+				(font
+					(size 1.27 1.27)
+				)
+				(justify right)
+			)
+		)
+		(property "Value" "SolderJumper_2_Open"
+			(at 262.89 228.092 90)
+			(effects
+				(font
+					(size 1.27 1.27)
+				)
+				(justify right)
+			)
+		)
+		(property "Footprint" "Jumper:SolderJumper-2_P1.3mm_Open_Pad1.0x1.5mm"
+			(at 271.78 218.44 0)
+			(effects
+				(font
+					(size 1.27 1.27)
+				)
+				(hide yes)
+			)
+		)
+		(property "Datasheet" "~"
+			(at 271.78 218.44 0)
+			(effects
+				(font
+					(size 1.27 1.27)
+				)
+				(hide yes)
+			)
+		)
+		(property "Description" "Solder Jumper, 2-pole, open"
+			(at 271.78 218.44 0)
+			(effects
+				(font
+					(size 1.27 1.27)
+				)
+				(hide yes)
+			)
+		)
+		(pin "1"
+		)
+		(pin "2"
+		)
+		(instances
+			(project ""
+				(path "/05d12b30-c3b1-455d-b907-9e9d56cc8f30/9caf0d13-589a-469d-9b5c-d69632aa737b"
+					(reference "JP1")
+					(unit 1)
+				)
+			)
+		)
+	)
+	(symbol
 		(lib_id "power:GND")
 		(at 85.09 71.12 0)
@@
 		(in_bom yes)
 		(on_board yes)
-		(dnp no)
+		(dnp yes)
 		(fields_autoplaced yes)
 		(property "Reference" "U7"
@@
 		(in_bom yes)
 		(on_board yes)
-		(dnp no)
+		(dnp yes)
 		(property "Reference" "D8"
 			(at 199.39 60.9599 90)
@@
 		(in_bom yes)
 		(on_board yes)
-		(dnp no)
+		(dnp yes)
 		(fields_autoplaced yes)
 		(property "Reference" "#PWR044"
@@
 					(unit 1)
 				)
+			)
+		)
+	)
+	(symbol
+		(lib_id "Jumper:SolderJumper_2_Open")
+		(at 276.86 218.44 90)
+		(unit 1)
+		(exclude_from_sim no)
+		(in_bom no)
+		(on_board yes)
+		(dnp no)
+		(property "Reference" "JP7"
+			(at 267.97 230.632 90)
+			(effects
+				(font
+					(size 1.27 1.27)
+				)
+				(justify right)
+			)
+		)
+		(property "Value" "SolderJumper_2_Open"
+			(at 267.97 228.092 90)
+			(effects
+				(font
+					(size 1.27 1.27)
+				)
+				(justify right)
+			)
+		)
+		(property "Footprint" "Jumper:SolderJumper-2_P1.3mm_Open_Pad1.0x1.5mm"
+			(at 276.86 218.44 0)
+			(effects
+				(font
+					(size 1.27 1.27)
+				)
+				(hide yes)
+			)
+		)
+		(property "Datasheet" "~"
+			(at 276.86 218.44 0)
+			(effects
+				(font
+					(size 1.27 1.27)
+				)
+				(hide yes)
+			)
+		)
+		(property "Description" "Solder Jumper, 2-pole, open"
+			(at 276.86 218.44 0)
+			(effects
+				(font
+					(size 1.27 1.27)
+				)
+				(hide yes)
+			)
+		)
+		(pin "1"
+		)
+		(pin "2"
+		)
+		(instances
+			(project "vectrix-vehicleman-0"
+				(path "/05d12b30-c3b1-455d-b907-9e9d56cc8f30/9caf0d13-589a-469d-9b5c-d69632aa737b"
+					(reference "JP7")
+					(unit 1)
+				)

Commit message: bom cleanup
Parts:
- D8: LCSC (none) -> C148219
- FB3: LCSC C96995 -> C85831
- U3: LCSC (none) -> C5350187
Changed lines of the file:
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@@
+			)
+		)
+		(property "LCSC" "C148219"
+			(at 201.93 62.23 90)
+			(effects
+				(font
+					(size 1.27 1.27)
+				)
+				(hide yes)
 			)
 		)
@@
 			)
 		)
-		(property "LCSC" "C96995"
+		(property "LCSC" " C85831"
 			(at 212.09 207.01 0)
 			(effects
@@
 			(at 85.09 58.42 0)
 			(effects
+				(font
+					(size 1.27 1.27)
+				)
+				(hide yes)
+			)
+		)
+		(property "LCSC" "C5350187"
+			(at 85.09 58.42 0)
+			(effects
