File: kicad/LTE.kicad_sch (KiCad schematic)
At the start: 0 parts

Commit message: WIP
Parts:
- added J8: SIM_Card_Shielded, Connector_Card:nanoSIM_Hinged_CUI_NSIM-2-C, symbol Connector:SIM_Card_Shielded
- added U18: SIM7070G, vehicle-manager:SIM7070G, symbol vehicle-manager:SIM7070G
Connections:
- new net: U18.16 (NC), U18.26 (NC), U18.35 (NC), U18.36 (NC), U18.40 (NC), U18.41 (NC), U18.42 (NC), U18.43 (NC), U18.44 (NC), U18.47 (NC), U18.51 (NC)
- new net: U18.55 (VBAT), U18.56 (VBAT), U18.57 (VBAT)
- new net GND: J8.SH, U18.17 (GND), U18.18 (GND), U18.2 (GND), U18.29 (GND), U18.39 (GND), U18.45 (GND), U18.46 (GND), U18.54 (GND), U18.58 (GND), U18.59 (GND), U18.61 (GND), U18.62 (GND), U18.63 (GND), U18.64 (GND), U18.65 (GND)

Commit message: sch done-ish
Parts:
- added C30, C71, C90, C94, C96: 10u 50V, Capacitor_SMD:C_1206_3216Metric, symbol Device:C
- added C70: 100uF 25V, Capacitor_SMD:CP_Elec_6.3x7.7, symbol Device:C_Polarized
- added C79, C80, C81, C91, C92, C93: 33pF 0603, Capacitor_SMD:C_0603_1608Metric, symbol Device:C
- added C85, C86, C87, C88, C89, C97, C98: 100nF 50V, Capacitor_SMD:C_0603_1608Metric, symbol Device:C
- added D1: TPESD1P0RFW, Package_TO_SOT_SMD:SOT-323_SC-70, symbol Power_Protection:SP0502BAJT
- added D18: LED GREEN, LED_SMD:LED_0805_2012Metric, symbol Device:LED
- added D19: LED PINK, LED_SMD:LED_0805_2012Metric, symbol Device:LED
- added D26: PESD5V0L4UG, Package_TO_SOT_SMD:SOT-353_SC-70-5, symbol Power_Protection:PESD5V0L4UG
- added FB4, FB5: FB_100R_2.5A, Inductor_SMD:L_0603_1608Metric, symbol Skrubis:FB_100R_2.5A
- added J10: GPS U.FL, Connector_Coaxial:U.FL_Hirose_U.FL-R-SMT-1_Vertical, symbol Connector:Conn_Coaxial
- added J11: LTE U.FL, Connector_Coaxial:U.FL_Hirose_U.FL-R-SMT-1_Vertical, symbol Connector:Conn_Coaxial
- added L1, L6, L7: 27nH, Inductor_SMD:L_0603_1608Metric, symbol Device:L
- added Q12, Q13, Q14, Q15, Q18: MMBT3904, Package_TO_SOT_SMD:SOT-23, symbol Transistor_BJT:MMBT3904
- added R104, R125, R126, R8, R96, R97: R_27R_0603, Resistor_SMD:R_0603_1608Metric, symbol Skrubis:R_27R_0603
- added R106, R118, R121, R122, R127, R128, R129, R132: 0R 0603, Resistor_SMD:R_0603_1608Metric, symbol Device:R
- added R107, R115, R116, R117, R119, R120, R123, R130, R131, R133, R134, R135: 4k7 0603, Resistor_SMD:R_0603_1608Metric, symbol Device:R
- added R124, R70, R71: 100k 0603, Resistor_SMD:R_0603_1608Metric, symbol Device:R
- added R43, R67: 1k 0603, Resistor_SMD:R_0603_1608Metric, symbol Device:R
- added TP1, TP2, TP3: TestPoint, TestPoint:TestPoint_Pad_D1.0mm, symbol Connector:TestPoint
- added U23: ME6217C33M5G, Package_TO_SOT_SMD:SOT-23-5, symbol Regulator_Linear:ME6211C33M5
Connections:
- net +1V8: now also U18.15 (VDD_EXT), C94.1, C96.1, C97.1, C98.1, R115.1, R116.1, R117.1, R119.1, R120.1, R123.1, R135.2
- net GND: now also J8.5 (GND), C30.2, C70.2, C71.2, C79.2, C80.2, C81.2, C85.2, C86.2, C87.2, C88.2, C89.2, C90.2, C92.1, C93.1, C94.2, C96.2, C97.2, C98.2, D1.3 (A), D26.2 (A), J10.2 (Ext), J11.2 (Ext), L6.2, L7.2, Q15.2 (E), R124.2, R130.1, R134.1, R43.2, R67.2, U23.2 (V_{SS})
- net at J8.1 (VCC): now also R8.1
- net at J8.2 (RST): now also D26.3 (K2), R96.1
- net at J8.3 (CLK): now also R97.1
- net at J8.7 (I/O): now also C81.1, D26.4 (K3), R104.1
- net at U18.1 (PWRKEY): now also R132.1
- net at U18.10 (UART1_RXD): now also R121.1
- net at U18.22 (DEBUG_RXD): now also TP2.1
- net at U18.23 (DEBUG_TXD): now also TP3.1
- net LTE_USB_VBUS_DET: now reaches U18.24 (USB_VBUS)
- net USB_LTE_DP: now reaches U18.27 (USB_DP)
- net USB_LTE_DN: now reaches U18.28 (USB_DM)
- net at U18.3 (UART1_DTR): now also R118.1
- net SIM_VDD: now reaches U18.30 (SIM_VDD)
- net SIM_VDD: now also D26.5 (K4), R8.2
- net SIM_DATA: now reaches U18.31 (SIM_DATA)
- net SIM_DATA: now also R104.2
- net SIM_CLK: now reaches U18.32 (SIM_CLK)
- net SIM_CLK: now also C79.1, D26.1 (K1), R97.2
- net SIM_RST: now reaches U18.33 (SIM_RST)
- net SIM_RST: now also C80.1, R96.2
- net LTE_GPIO5: now reaches U18.48 (GPIO5/SPI_CS)
- net LTE_GPIO5: now also Q18.2 (E), Q18.3 (C), R133.2, R134.2, R135.1
- net at U18.52 (NETLIGHT): now also D19.2 (A)
- net GNSS_ANT: now reaches U18.53 (GNSS_ANT)
- net GNSS_ANT: now also L7.1, R127.2
- net at U18.55 (VBAT), U18.56 (VBAT), U18.57 (VBAT): now also C30.1, C70.1, C85.1, C86.1, C87.1, FB4.1, R106.1
- net at U18.6 (BOOT_CFG): now also TP1.1
- net LTE_ANT: now reaches U18.60 (RF_ANT)
- net LTE_ANT: now also R129.2
- net at U18.66 (STATUS): now also D18.2 (A)
- net at U18.9 (UART1_TXD): now also R122.1
- new net: C89.1, C90.1, FB5.2, U23.1 (V_{IN})
- new net: D18.1 (K), R43.1
- new net: C92.2, D1.1 (K), J11.1 (In), R128.1
- new net: D19.1 (K), R67.1
- new net: C91.1, L6.1, R127.1
- new net: Q14.1 (B), R119.2
- new net: Q15.1 (B), R130.2, R131.2
- new net: C93.2, R128.2, R129.1
- new net: L1.2, R125.2, R126.2
- new net: Q13.1 (B), R116.2
- new net: Q12.1 (B), R115.2
- new net: C91.2, J10.1 (In), L1.1
- new net: Q18.1 (B), R123.2
- new net +3V3: R106.2, R107.1, R133.1, R70.1, R71.1
- new net GPS_LDO_EN: R124.1, U23.3 (CE)
- new net GPS_VCC: C71.1, C88.1, R125.1, R126.1, U23.5 (V_{OUT})
- new net LTE_DTR: Q14.2 (E), R71.2
- new net LTE_POWERKEY: R131.1
- new net LTE_RX: Q13.2 (E), R70.2
- new net LTE_TX: Q12.3 (C), R107.2
- new net POWERKEY: Q15.3 (C), R132.2
- new net UART1_DTR: Q14.3 (C), R118.2, R120.2
- new net UART1_RXD: Q13.3 (C), R117.2, R121.2
- new net UART1_TXD: Q12.2 (E), R122.2
- new net VBUS: FB4.2, FB5.1
- no-connect marks 0 -> 20
Other:
- company: (none) -> ©CC-BY-NC
- title: (none) -> VehicleMan

Commit message: WIP
Parts:
- removed C91, C92: 33pF 0603, Capacitor_SMD:C_0603_1608Metric, symbol Device:C
- removed C97: 100nF 50V, Capacitor_SMD:C_0603_1608Metric, symbol Device:C
- removed R125, R126: R_27R_0603, Resistor_SMD:R_0603_1608Metric, symbol Skrubis:R_27R_0603
- removed R127: 0R 0603, Resistor_SMD:R_0603_1608Metric, symbol Device:R
- added C95: 33pF 0402, Capacitor_SMD:C_0402_1005Metric, symbol Device:C
- added R143: 0R 0402, Resistor_SMD:R_0402_1005Metric, symbol Device:R
- added R144: 10R 0402, Resistor_SMD:R_0402_1005Metric, symbol Device:R
- C93: value 33pF 0603 -> 33pF 0402; footprint Capacitor_SMD:C_0603_1608Metric -> Capacitor_SMD:C_0402_1005Metric; LCSC C107047 -> C1562
- C96: value 10u 50V -> 33pF 0402; footprint Capacitor_SMD:C_1206_3216Metric -> Capacitor_SMD:C_0402_1005Metric; LCSC C13585 -> C1562
- L1: value 27nH -> 47nH; footprint Inductor_SMD:L_0603_1608Metric -> Inductor_SMD:L_0402_1005Metric; LCSC C90208 -> C97998
- L6, L7: footprint Inductor_SMD:L_0603_1608Metric -> Inductor_SMD:L_0402_1005Metric; LCSC C90208 -> C12669
- R128, R129: value 0R 0603 -> 0R 0402; footprint Resistor_SMD:R_0603_1608Metric -> Resistor_SMD:R_0402_1005Metric; LCSC C21189 -> C106231
Connections:
- net +1V8: no longer C96.1
- net GND: now also C95.1; no longer C96.2
- net GNSS_ANT: now also L6.1, R143.2; no longer L7.1
- net GPS_VCC: now also R144.2
- net SIM_CLK: now also D26.3 (K2); no longer D26.1 (K1)
- net SIM_RST: now also D26.1 (K1)
- net at D1.1 (K), J11.1 (In), R128.1: now also D1.2 (K), C95.2
- net at L1.2: now also R144.1
- net at J10.1 (In), L1.1: now also C96.1
- net at J8.2 (RST), R96.1: no longer D26.3 (K2)
- new net: C96.2, L7.1, R143.1

Commit message: WIP
Parts:
- removed C85, C86: 100nF 50V, Capacitor_SMD:C_0603_1608Metric, symbol Device:C
- added C100: Tant 47u 17V, Capacitor_Tantalum_SMD:CP_EIA-3528-12_Kemet-T, symbol Device:C_Polarized
- C70: value 100uF 25V -> Tant 47u 17V; footprint Capacitor_SMD:CP_Elec_6.3x7.7 -> Capacitor_Tantalum_SMD:CP_EIA-3528-12_Kemet-T; LCSC C2918360 -> C136751
Connections:
- net GND: now also C100.2
- net LTE_GPIO5: no longer Q18.3 (C), R133.2
- net SIM_CLK: no longer D26.3 (K2)
- net SIM_RST: no longer D26.1 (K1)
- net SIM_VDD: no longer D26.5 (K4)
- net at C30.1, C70.1, C87.1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: now also C100.1
- net at J8.3 (CLK), R97.1: now also D26.3 (K2)
- net at J8.1 (VCC), R8.1: now also D26.5 (K4)
- net at J8.2 (RST), R96.1: now also D26.1 (K1)
- new net LTE_GPIO5_HV: Q18.3 (C), R133.2
Other:
- moved on the sheet: C30, C70, C87, FB4

Commit message: R0
Connections:
- net at C81.1, J8.7 (I/O), R104.1: no longer D26.4 (K3)
Changed lines of the file:
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@@
 	)
 	(junction
-		(at 68.58 177.8)
-		(diameter 0)
-		(color 0 0 0 0)
-	)
-	(junction
 		(at 256.54 146.05)
 		(diameter 0)
@@
 	(wire
 		(pts
-			(xy 68.58 177.8) (xy 85.09 177.8)
-		)
-		(stroke
-			(width 0)
-			(type default)
-		)
-	)
-	(wire
-		(pts
 			(xy 160.02 170.18) (xy 154.94 170.18)
 		)
@@
 	(wire
 		(pts
-			(xy 60.96 177.8) (xy 68.58 177.8)
+			(xy 60.96 177.8) (xy 85.09 177.8)
 		)
 		(stroke
@@
 	(symbol
 		(lib_id "Power_Protection:PESD5V0L4UG")
-		(at 68.58 175.26 270)
-		(mirror x)
-		(unit 3)
-		(exclude_from_sim no)
-		(in_bom yes)
-		(on_board yes)
-		(dnp no)
-		(property "Reference" "D26"
-			(at 71.12 176.5301 90)
-			(effects
-				(font
-					(size 1.27 1.27)
-				)
-				(justify left)
-			)
-		)
-		(property "Value" "PESD5V0L4UG"
-			(at 71.12 173.9901 90)
-			(effects
-				(font
-					(size 1.27 1.27)
-				)
-				(justify left)
-			)
-		)
-		(property "Footprint" "Package_TO_SOT_SMD:SOT-353_SC-70-5"
-			(at 73.66 175.26 0)
-			(effects
-				(font
-					(size 1.27 1.27)
-				)
-				(hide yes)
-			)
-		)
-		(property "Datasheet" "https://assets.nexperia.com/documents/data-sheet/PESDXL4UF_G_W.pdf"
-			(at 63.5 175.26 0)
-			(effects
-				(font
-					(size 1.27 1.27)
-				)
-				(hide yes)
-			)
-		)
-		(property "Description" "Low capacitance unidirectional quadruple ESD protection diode array, 5.0V, Common Anode, SOT-353"
-			(at 68.58 175.26 0)
-			(effects
-				(font
-					(size 1.27 1.27)
-				)
-				(hide yes)
-			)
-		)
-		(property "LCSC" "C5116450"
-			(at 68.58 175.26 90)
-			(effects
-				(font
-					(size 1.27 1.27)
-				)
-				(hide yes)
-			)
-		)
-		(pin "1"
-		)
-		(pin "4"
-		)
-		(pin "2"
-		)
-		(pin "3"
-		)
-		(pin "5"
-		)
-		(instances
-			(project "vectrix-vehicleman-0"
-				(path "/05d12b30-c3b1-455d-b907-9e9d56cc8f30/99782543-f9fb-4dd7-a2c0-0df378ed7ddd"
-					(reference "D26")
-					(unit 3)
-				)
-			)
-		)
-	)
-	(symbol
-		(lib_id "Power_Protection:PESD5V0L4UG")
 		(at 85.09 161.29 90)
 		(unit 1)
@@
 				)
 			)
+		)
+	)
+	(symbol
+		(lib_id "Power_Protection:PESD5V0L4UG")
+		(at 116.84 153.67 270)
+		(mirror x)
+		(unit 3)
+		(exclude_from_sim no)
+		(in_bom yes)
+		(on_board yes)
+		(dnp no)
+		(property "Reference" "D26"
+			(at 119.38 154.9401 90)
+			(effects
+				(font
+					(size 1.27 1.27)
+				)
+				(justify left)
+			)
+		)
+		(property "Value" "PESD5V0L4UG"
+			(at 119.38 152.4001 90)
+			(effects
+				(font
+					(size 1.27 1.27)
+				)
+				(justify left)
+			)
+		)
+		(property "Footprint" "Package_TO_SOT_SMD:SOT-353_SC-70-5"
+			(at 121.92 153.67 0)
+			(effects
+				(font
+					(size 1.27 1.27)
+				)
+				(hide yes)
+			)
+		)
+		(property "Datasheet" "https://assets.nexperia.com/documents/data-sheet/PESDXL4UF_G_W.pdf"
+			(at 111.76 153.67 0)
+			(effects
+				(font
+					(size 1.27 1.27)
+				)
+				(hide yes)
+			)
+		)
+		(property "Description" "Low capacitance unidirectional quadruple ESD protection diode array, 5.0V, Common Anode, SOT-353"
+			(at 116.84 153.67 0)
+			(effects
+				(font
+					(size 1.27 1.27)
+				)
+				(hide yes)
+			)
+		)
+		(property "LCSC" "C5116450"
+			(at 116.84 153.67 90)
+			(effects
+				(font
+					(size 1.27 1.27)
+				)
+				(hide yes)
+			)
+		)
+		(pin "1"
+		)
+		(pin "4"
+		)
+		(pin "2"
+		)
+		(pin "3"
+		)
+		(pin "5"
+		)
+		(instances
+			(project "vectrix-vehicleman-0"
+				(path "/05d12b30-c3b1-455d-b907-9e9d56cc8f30/99782543-f9fb-4dd7-a2c0-0df378ed7ddd"
+					(reference "D26")
+					(unit 3)
+				)
+			)

Commit message: bom cleanup
Parts:
- FB4, FB5: LCSC C96995 -> C85831
- J10: value GPS U.FL -> u.fl
- J11: value LTE U.FL -> u.fl
- Q12, Q13, Q14, Q15, Q18: LCSC (none) -> C20526
Changed lines of the file:
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@@
 			)
 		)
-		(property "Value" "LTE U.FL"
+		(property "Value" "u.fl"
 			(at 276.86 139.9931 0)
 			(effects
@@
 			)
 		)
+		(property "LCSC" "C20526"
+			(at 35.56 87.63 0)
+			(effects
+				(font
+					(size 1.27 1.27)
+				)
+				(hide yes)
+			)
+		)
 		(pin "1"
 		)
@@
 			)
 		)
+		(property "LCSC" "C20526"
+			(at 48.26 119.38 0)
+			(effects
+				(font
+					(size 1.27 1.27)
+				)
+				(hide yes)
+			)
+		)
 		(pin "1"
 		)
@@
 			)
 		)
-		(property "LCSC" "C96995"
+		(property "LCSC" " C85831"
 			(at 200.66 22.86 0)
 			(effects
@@
 			)
 		)
-		(property "LCSC" "C96995"
+		(property "LCSC" " C85831"
 			(at 191.77 44.45 0)
 			(effects
@@
 			)
 		)
+		(property "LCSC" "C20526"
+			(at 88.9 119.38 0)
+			(effects
+				(font
+					(size 1.27 1.27)
+				)
+				(hide yes)
+			)
+		)
 		(pin "1"
 		)
@@
 			)
 		)
-		(property "Value" "GPS U.FL"
+		(property "Value" "u.fl"
 			(at 267.97 72.6831 0)
 			(effects
@@
 			)
 		)
+		(property "LCSC" "C20526"
+			(at 76.2 44.45 0)
+			(effects
+				(font
+					(size 1.27 1.27)
+				)
+				(hide yes)
+			)
+		)
 		(pin "1"
 		)
@@
 			(at 35.56 44.45 0)
 			(effects
+				(font
+					(size 1.27 1.27)
+				)
+				(hide yes)
+			)
+		)
+		(property "LCSC" "C20526"
+			(at 35.56 44.45 0)
+			(effects
