File: kicad/switches.kicad_sch (KiCad schematic)
At the start: 0 parts

Commit message: sch done-ish
Parts:
- added D29, D30, D31, D32, D33, D34, D35, D36: 1N4001, Diode_SMD:D_SMA, symbol Diode:1N4001
- added F10, F11, F12, F13, F14, F15: Polyfuse 1.5A, Fuse:Fuse_1812_4532Metric, symbol Device:Polyfuse
- added F32, F33: 200mA PTC, Fuse:Fuse_0805_2012Metric, symbol Device:Polyfuse
- added J13: K1, TerminalBlock_Phoenix:TerminalBlock_Phoenix_MKDS-1,5-3-5.08_1x03_P5.08mm_Horizontal, symbol Connector:Screw_Terminal_01x03
- added J14: K1, TerminalBlock_Phoenix:TerminalBlock_Phoenix_MKDS-1,5-2-5.08_1x02_P5.08mm_Horizontal, symbol Connector:Screw_Terminal_01x02
- added J15: K2, TerminalBlock_Phoenix:TerminalBlock_Phoenix_MKDS-1,5-2-5.08_1x02_P5.08mm_Horizontal, symbol Connector:Screw_Terminal_01x02
- added J16: K2, TerminalBlock_Phoenix:TerminalBlock_Phoenix_MKDS-1,5-3-5.08_1x03_P5.08mm_Horizontal, symbol Connector:Screw_Terminal_01x03
- added K1, K2: G2RL-24 DC5, Relay_THT:Relay_DPDT_Omron_G2RL-2, symbol Relay:G2RL-2
- added Q16, Q17: Q_NPN_BEC, Package_TO_SOT_SMD:SOT-23, symbol Device:Q_NPN_BEC
- added Q19, Q20, Q21, Q22: PMOS_30V_5.5A, Package_TO_SOT_SMD:SOT-23, symbol Skrubis:Q_PMOS_30V_5.5A_SOT23
- added R105, R140, R141, R142: 10k 0603, Resistor_SMD:R_0603_1608Metric, symbol Device:R
- added R136, R138: 4k7 0603, Resistor_SMD:R_0603_1608Metric, symbol Device:R
- added R137, R139: 1.2k 0603, Resistor_SMD:R_0603_1608Metric, symbol Device:R
- added R161, R162, R163, R164: 470R 0603, Resistor_SMD:R_0603_1608Metric, symbol Device:R
Connections:
- new net: Q20.1 (G), R140.2, R162.1
- new net: F13.1, Q20.2 (S)
- new net: D30.1 (K), J14.1 (Pin_1), K1.14
- new net: Q16.1 (B), R136.2, R137.1
- new net: Q17.1 (B), R138.2, R139.1
- new net: D32.1 (K), J15.1 (Pin_1), K2.14
- new net: Q19.1 (G), R105.2, R161.1
- new net: Q21.1 (G), R141.2, R163.1
- new net: Q22.1 (G), R142.2, R164.1
- new net: D31.1 (K), F33.1, K2.A1
- new net: D31.2 (A), K2.A2, Q17.3 (C)
- new net: F11.2, K2.11
- new net: J16.3 (Pin_3), K2.21
- new net: J16.1 (Pin_1), K2.22
- new net: J16.2 (Pin_2), K2.24
- new net: F14.1, Q21.2 (S)
- new net: F10.2, K1.11
- new net: F12.1, Q19.2 (S)
- new net: D29.1 (K), F32.1, K1.A1
- new net: D29.2 (A), K1.A2, Q16.3 (C)
- new net: F15.1, Q22.2 (S)
- new net: J13.3 (Pin_3), K1.21
- new net: J13.1 (Pin_1), K1.22
- new net: J13.2 (Pin_2), K1.24
- new net +12V: F10.1, F11.1, F12.2, F13.2, F14.2, F15.2, R105.1, R140.1, R141.1, R142.1
- new net GND: D30.2 (A), D32.2 (A), D33.2 (A), D34.2 (A), D35.2 (A), D36.2 (A), J14.2 (Pin_2), J15.2 (Pin_2), Q16.2 (E), Q17.2 (E), R137.2, R139.2
- new net RELAY_1_GPIO: R136.1
- new net RELAY_2_GPIO: R138.1
- new net SW1: R161.2
- new net SW1-OUT: D33.1 (K), Q19.3 (D)
- new net SW2: R162.2
- new net SW2-OUT: D34.1 (K), Q20.3 (D)
- new net SW3: R163.2
- new net SW3-OUT: D35.1 (K), Q21.3 (D)
- new net SW4: R164.2
- new net SW4-OUT: D36.1 (K), Q22.3 (D)
- new net VBUS: F32.2, F33.2
- no-connect marks 0 -> 2
Other:
- note added: "1-24V 2-GND"
- note added: "1-NC 2-NO 3-COM"
- company: (none) -> ©CC-BY-NC
- title: (none) -> VehicleMan

Commit message: WIP
Parts:
- removed J13: K1, TerminalBlock_Phoenix:TerminalBlock_Phoenix_MKDS-1,5-3-5.08_1x03_P5.08mm_Horizontal, symbol Connector:Screw_Terminal_01x03
- removed J14: K1, TerminalBlock_Phoenix:TerminalBlock_Phoenix_MKDS-1,5-2-5.08_1x02_P5.08mm_Horizontal, symbol Connector:Screw_Terminal_01x02
- removed J15: K2, TerminalBlock_Phoenix:TerminalBlock_Phoenix_MKDS-1,5-2-5.08_1x02_P5.08mm_Horizontal, symbol Connector:Screw_Terminal_01x02
- removed J16: K2, TerminalBlock_Phoenix:TerminalBlock_Phoenix_MKDS-1,5-3-5.08_1x03_P5.08mm_Horizontal, symbol Connector:Screw_Terminal_01x03
- added J25: K1, TerminalBlock_4Ucon:TerminalBlock_4Ucon_1x03_P3.50mm_Horizontal, symbol Connector:Screw_Terminal_01x03
- added J26: K1, TerminalBlock_4Ucon:TerminalBlock_4Ucon_1x02_P3.50mm_Horizontal, symbol Connector:Screw_Terminal_01x02
- added J27: K2, TerminalBlock_4Ucon:TerminalBlock_4Ucon_1x03_P3.50mm_Horizontal, symbol Connector:Screw_Terminal_01x03
- added J28: K2, TerminalBlock_4Ucon:TerminalBlock_4Ucon_1x02_P3.50mm_Horizontal, symbol Connector:Screw_Terminal_01x02
- K1, K2: now fitted
Connections:
- net GND: now also J26.2 (Pin_2), J28.2 (Pin_2)
- net at D30.1 (K), K1.14: now also J26.1 (Pin_1)
- net at D32.1 (K), K2.14: now also J28.1 (Pin_1)
- net at K2.21: now also J27.3 (Pin_3)
- net at K2.22: now also J27.1 (Pin_1)
- net at K2.24: now also J27.2 (Pin_2)
- net at K1.21: now also J25.3 (Pin_3)
- net at K1.22: now also J25.1 (Pin_1)
- net at K1.24: now also J25.2 (Pin_2)

Commit message: WIP
Parts:
- removed D33, D34, D35, D36: 1N4001, Diode_SMD:D_SMA, symbol Diode:1N4001

Commit message: bom cleanup
Parts:
- J25: value K1 -> Screwterminal 01x03
- J26: value K1 -> Screwterminal 01x02
- J27: value K2 -> Screwterminal 01x03
- J28: value K2 -> Screwterminal 01x02
Changed lines of the file:
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@@
 			)
 		)
-		(property "Value" "K2"
+		(property "Value" "Screwterminal 01x02"
 			(at 255.27 86.36 0)
 			(effects
@@
 			)
 		)
-		(property "Value" "K1"
+		(property "Value" "Screwterminal 01x02"
 			(at 256.54 29.21 0)
 			(effects
@@
 			)
 		)
-		(property "Value" "K1"
+		(property "Value" "Screwterminal 01x03"
 			(at 256.54 57.15 0)
 			(effects
@@
 			)
 		)
-		(property "Value" "K2"
+		(property "Value" "Screwterminal 01x03"
 			(at 255.27 114.3 0)
 			(effects
