File: kicad/type2.kicad_sch (KiCad schematic)
At the start: 27 parts, among them Q10 BSS138-7-F, Q11 BSS138-7-F, Q5 BSS138-7-F, Q9 BSS138-7-F, U20 LM321

Commit message: bom cleanup
Parts:
- Q10, Q11, Q5, Q9: LCSC C40912 -> C112239
Changed lines of the file:
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@@
 			)
 		)
-		(property "LCSC" "C40912"
+		(property "LCSC" "C112239"
 			(at 116.84 91.44 0)
 			(effects
@@
 			)
 		)
-		(property "LCSC" "C40912"
+		(property "LCSC" "C112239"
 			(at 133.35 91.44 0)
 			(effects
@@
 			)
 		)
-		(property "LCSC" "C40912"
+		(property "LCSC" "C112239"
 			(at 82.55 91.44 0)
 			(effects
@@
 			)
 		)
-		(property "LCSC" "C40912"
+		(property "LCSC" "C112239"
 			(at 100.33 91.44 0)
 			(effects
